File: pcb/pcb.kicad_pcb (KiCad board)
At the start: 2 copper layers, 94.3 x 83.3 mm, 10 parts

Commit message: Updates
Parts:
- CAPACITOR_1, CAPACITOR_2: footprint Capacitor_THT:CP_Radial_D5.0mm_P2.00mm -> Capacitor_THT:CP_Radial_D4.0mm_P2.00mm
- MPU_SENSOR_1: footprint GY-521:MODULE_GY-521 -> SelfBalancingRobot:MODULE_GY-521
