File: pcb/pcb.kicad_sch (KiCad schematic)
At the start: 10 parts

Commit message: Updates
Parts:
- CAPACITOR_1, CAPACITOR_2: footprint Capacitor_THT:CP_Radial_D5.0mm_P2.00mm -> Capacitor_THT:CP_Radial_D4.0mm_P2.00mm
- MPU_SENSOR_1: footprint GY-521:MODULE_GY-521 -> SelfBalancingRobot:MODULE_GY-521
Connections:
- net GND: now also MPU_SENSOR_1.GND; no longer MPU_SENSOR_1.2 (GND)
- net at BUCKCONVERTER_1.4 (3v3), ESP_32.16 (Pin_16), MOTOR_DRV1.5 (Pin_5)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: now also MPU_SENSOR_1.VCC; no longer MPU_SENSOR_1.1 (VCC)
- net at ESP_32.29 (Pin_29): now also MPU_SENSOR_1.SCL; no longer MPU_SENSOR_1.3 (SCL)
- net at ESP_32.26 (Pin_26): now also MPU_SENSOR_1.SDA; no longer MPU_SENSOR_1.4 (SDA)
Changed lines of the file:
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@@
 			)
 		)
-		(property "Footprint" "GY-521:MODULE_GY-521"
+		(property "Footprint" "SelfBalancingRobot:MODULE_GY-521"
 			(at 176.53 73.66 0)
 			(hide yes)
@@
 			)
 		)
-		(pin "8"
-		)
-		(pin "1"
-		)
-		(pin "3"
-		)
-		(pin "4"
-		)
-		(pin "5"
-		)
-		(pin "6"
-		)
-		(pin "7"
-		)
-		(pin "2"
+		(pin "AD0"
+		)
+		(pin "SDA"
+		)
+		(pin "XCL"
+		)
+		(pin "VCC"
+		)
+		(pin "SCL"
+		)
+		(pin "XDA"
+		)
+		(pin "GND"
+		)
+		(pin "INT"
 		)
 		(instances
@@
 			)
 		)
-		(property "Footprint" "Capacitor_THT:CP_Radial_D5.0mm_P2.00mm"
+		(property "Footprint" "Capacitor_THT:CP_Radial_D4.0mm_P2.00mm"
 			(at 192.7352 114.3 0)
 			(hide yes)
@@
 			)
 		)
-		(property "Footprint" "Capacitor_THT:CP_Radial_D5.0mm_P2.00mm"
+		(property "Footprint" "Capacitor_THT:CP_Radial_D4.0mm_P2.00mm"
 			(at 187.6552 139.7 0)
 			(hide yes)
